File: KiCad Data/General_BNC_PCB_BOARD2.kicad_sch (KiCad schematic)
At the start: 16 parts, among them P1 Potentiometer, Digikey P/N: 3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

Commit message: Add files via upload
Parts:
- added TP2: TestPoint, GENERAL PROJECT - NUMBER 1 LIBRARY - FOOTPRINTS:TestPoint, symbol Connector:TestPoint
Connections:
- net GND: now also IDC1.14 (G), IDC1.7 (C), TP2.1; no longer IDC1.1 (C), IDC1.8 (G)
- net at BNC2.1 (In): now also IDC1.9 (G); no longer IDC1.10 (G)
- net at BNC2.2 (Ext): now also IDC1.2 (C); no longer IDC1.3 (C)
- net at BNC5.1 (In): now also IDC1.12 (G); no longer IDC1.13 (G)
- net at BNC5.2 (Ext): now also IDC1.5 (C); no longer IDC1.6 (C)
- net at BNC4.1 (In): now also IDC1.11 (G); no longer IDC1.12 (G)
- net at BNC4.2 (Ext): now also IDC1.4 (C); no longer IDC1.5 (C)
- net at BNC3.1 (In): now also IDC1.10 (G); no longer IDC1.11 (G)
- net at BNC3.2 (Ext): now also IDC1.3 (C); no longer IDC1.4 (C)
- net at BNC1.1 (In): now also IDC1.8 (G); no longer IDC1.9 (G)
- net at BNC1.2 (Ext): now also IDC1.1 (C); no longer IDC1.2 (C)
- net at BNC6.1 (In): now also IDC1.13 (G); no longer IDC1.14 (G)
- net at BNC6.2 (Ext): now also IDC1.6 (C); no longer IDC1.7 (C)
Other:
- moved on the sheet: IDC1
